Commit message: Bebop2 drone

File: xacro/bebop2.xacro (robot description, xacro)
@@ -5,5 +5,5 @@
   <xacro:property name="rotor_velocity_slowdown_sim" value="10" />
   <xacro:property name="use_mesh_file" value="true" />
-  <xacro:property name="mesh_file" value="package://rotors_description/meshes/bebop2.dae" />
+  <xacro:property name="mesh_file" value="package://bearings/meshes/bebop2.dae" />
   <xacro:property name="mass" value="0.503" /> <!-- [kg] -->
   <xacro:property name="body_width" value="0.316618" /> <!-- [m] -->
@@ -62,5 +62,5 @@
     color=""
     use_own_mesh="true"
-    mesh="package://rotors_description/meshes/propeller_fr.dae">
+    mesh="package://bearings/meshes/propeller_fr.dae">
     <origin xyz="0.08456 -0.11435 -0.00501" rpy="0 0 0" />
     <xacro:insert_block name="rotor_inertia" />
@@ -83,5 +83,5 @@
     color=""
     use_own_mesh="true"
-    mesh="package://rotors_description/meshes/propeller_rl.dae">
+    mesh="package://bearings/meshes/propeller_rl.dae">
     <origin xyz="-0.09035 0.11452 -0.00501" rpy="0 0 0" />
     <xacro:insert_block name="rotor_inertia" />
@@ -103,5 +103,5 @@
     color=""
     use_own_mesh="true"
-    mesh="package://rotors_description/meshes/propeller_fl.dae">
+    mesh="package://bearings/meshes/propeller_fl.dae">
     <origin xyz="0.08456 0.11463 -0.00501" rpy="0 0 0" />
     <xacro:insert_block name="rotor_inertia" />
@@ -123,5 +123,5 @@
     color=""
     use_own_mesh="true"
-    mesh="package://rotors_description/meshes/propeller_rr.dae">
+    mesh="package://bearings/meshes/propeller_rr.dae">
     <origin xyz="-0.09035 -0.11423 -0.00501" rpy="0 0 0" />
     <xacro:insert_block name="rotor_inertia" />

File: xacro/bebop2_base.xacro (robot description, xacro)
@@ -3,5 +3,5 @@
   <xacro:include filename="$(find rotors_description)/urdf/component_snippets.xacro" />
   <!-- Instantiate ardrone "mechanics" -->
-  <xacro:include filename="$(find rotors_description)/urdf/bebop2.xacro" />
+  <xacro:include filename="$(find bearings)/xacro/bebop2.xacro" />
   <!-- Instantiate a controller. -->
   <xacro:controller_plugin_macro namespace="${namespace}" imu_sub_topic="imu" />
