Commit message: Bebop2 drone

File: description/camera.xacro (robot description, xacro)
@@ -1,5 +1,5 @@
 <?xml version="1.0"?>
 <robot xmlns:xacro="http://www.ros.org/wiki/xacro">
-  <xacro:macro name="front_camera" params="namespace">
+  <xacro:macro name="camera_base" params="namespace">
     <joint name="camera_joint" type="fixed">
       <parent link="${namespace}/base_link"/>
@@ -63,5 +63,5 @@
     </gazebo>
   </xacro:macro>
-  <xacro:macro name="under_camera" params="namespace">
+  <xacro:macro name="camera_secondary" params="namespace">
     <joint name="camera_under_joint" type="fixed">
       <parent link="${namespace}/base_link"/>

Commit message: Added 5 drones

File: description/camera.xacro (robot description, xacro)
@@ -63,5 +63,5 @@
     </gazebo>
   </xacro:macro>
-  <xacro:macro name="camera_secondary" params="namespace">
+  <xacro:macro name="under_camera" params="namespace">
     <joint name="camera_under_joint" type="fixed">
       <parent link="${namespace}/base_link"/>

File: xacro/bebop2_1.xacro (robot description, xacro)
@@ -128,5 +128,5 @@
   </xacro:vertical_rotor>
  <!--Mount a Camera-->
-  <xacro:camera_macro
+  <!-- <xacro:camera_macro
       namespace="${namespace}"
       parent_link="${namespace}/base_link"
@@ -144,4 +144,6 @@
       <box size="0.001 0.001 0.001" />
       <origin xyz="0.1 0 0" rpy="0 0 0" />
-  </xacro:camera_macro>
+  </xacro:camera_macro> -->
+  <xacro:include filename="$(find bearings)/description/camera_bebop2.xacro"/>
+  <xacro:camera_base namespace="${namespace}" ></xacro:camera_base>
 </robot>

File: xacro/bebop2_2.xacro (robot description, xacro)
@@ -128,5 +128,5 @@
   </xacro:vertical_rotor>
  <!--Mount a Camera-->
-  <xacro:camera_macro
+  <!-- <xacro:camera_macro
       namespace="${namespace}"
       parent_link="${namespace}/base_link"
@@ -144,4 +144,6 @@
       <box size="0.001 0.001 0.001" />
       <origin xyz="0.1 0 0" rpy="0 0 0" />
-  </xacro:camera_macro>
+  </xacro:camera_macro> -->
+  <xacro:include filename="$(find bearings)/description/camera_bebop2.xacro"/>
+  <xacro:camera_base namespace="${namespace}" ></xacro:camera_base>
 </robot>

File: xacro/bebop2_3.xacro (robot description, xacro)
@@ -128,5 +128,5 @@
   </xacro:vertical_rotor>
  <!--Mount a Camera-->
-  <xacro:camera_macro
+  <!-- <xacro:camera_macro
       namespace="${namespace}"
       parent_link="${namespace}/base_link"
@@ -144,4 +144,6 @@
       <box size="0.001 0.001 0.001" />
       <origin xyz="0.1 0 0" rpy="0 0 0" />
-  </xacro:camera_macro>
+  </xacro:camera_macro> -->
+  <xacro:include filename="$(find bearings)/description/camera_bebop2.xacro"/>
+  <xacro:camera_base namespace="${namespace}" ></xacro:camera_base>
 </robot>

File: xacro/bebop2_4.xacro (robot description, xacro)
@@ -128,5 +128,5 @@
   </xacro:vertical_rotor>
  <!--Mount a Camera-->
-  <xacro:camera_macro
+  <!-- <xacro:camera_macro
       namespace="${namespace}"
       parent_link="${namespace}/base_link"
@@ -144,4 +144,6 @@
       <box size="0.001 0.001 0.001" />
       <origin xyz="0.1 0 0" rpy="0 0 0" />
-  </xacro:camera_macro>
+  </xacro:camera_macro> -->
+  <xacro:include filename="$(find bearings)/description/camera_bebop2.xacro"/>
+  <xacro:camera_base namespace="${namespace}" ></xacro:camera_base>
 </robot>

File: xacro/iris1.xacro (robot description, xacro)
@@ -165,5 +165,5 @@
   </xacro:camera_macro> -->
   <xacro:include filename="$(find bearings)/description/camera.xacro"/>
-  <xacro:front_camera namespace="${namespace}" ></xacro:front_camera>
+  <xacro:camera_base namespace="${namespace}" ></xacro:camera_base>
   <xacro:under_camera namespace="${namespace}" ></xacro:under_camera>
 </robot>

File: xacro/iris2.xacro (robot description, xacro)
@@ -165,5 +165,5 @@
   </xacro:camera_macro> -->
   <xacro:include filename="$(find bearings)/description/camera.xacro"/>
-  <xacro:front_camera namespace="${namespace}" ></xacro:front_camera>
+  <xacro:camera_base namespace="${namespace}" ></xacro:camera_base>
   <xacro:under_camera namespace="${namespace}" ></xacro:under_camera>
 </robot>

File: xacro/iris3.xacro (robot description, xacro)
@@ -168,5 +168,5 @@
   </xacro:camera_macro> -->
   <xacro:include filename="$(find bearings)/description/camera.xacro"/>
-  <xacro:front_camera namespace="${namespace}" ></xacro:front_camera>
+  <xacro:camera_base namespace="${namespace}" ></xacro:camera_base>
   <xacro:under_camera namespace="${namespace}" ></xacro:under_camera>
 </robot>

File: xacro/iris4.xacro (robot description, xacro)
@@ -168,5 +168,5 @@
   </xacro:camera_macro> -->
   <xacro:include filename="$(find bearings)/description/camera.xacro"/>
-  <xacro:front_camera namespace="${namespace}" ></xacro:front_camera>
+  <xacro:camera_base namespace="${namespace}" ></xacro:camera_base>
   <xacro:under_camera namespace="${namespace}" ></xacro:under_camera>
 </robot>

Commit message: Added 5 drones

File: description/camera.xacro (robot description, xacro)
@@ -10,5 +10,5 @@
       <visual>
         <geometry>
-          <box size="0.010 0.03 0.03"/>
+          <box size="0.001 0.001 0.001"/>
         </geometry>
         <material name="Red"/>
@@ -58,5 +58,5 @@
         <plugin name="camera_controller" filename="libgazebo_ros_camera.so">
           <frame_name>camera_link_optical</frame_name>
-          <cameraName>camera_front_camera</cameraName>
+          <cameraName>camera_base</cameraName>
         </plugin>
       </sensor>

File: description/camera_bebop2.xacro (robot description, xacro)
@@ -28,5 +28,5 @@
         <update_rate>30</update_rate>
         <camera>
-          <horizontal_fov>1.7</horizontal_fov>
+          <horizontal_fov>1.0472</horizontal_fov>
           <image>
             <width>856</width>
@@ -58,5 +58,5 @@
         <plugin name="camera_controller" filename="libgazebo_ros_camera.so">
           <frame_name>camera_link_optical</frame_name>
-          <cameraName>camera_front_camera</cameraName>
+          <cameraName>camera_base</cameraName>
         </plugin>
       </sensor>

File: xacro/bebop2_2.xacro (robot description, xacro)
@@ -128,5 +128,5 @@
   </xacro:vertical_rotor>
  <!--Mount a Camera-->
-  <!-- <xacro:camera_macro
+  <xacro:camera_macro
       namespace="${namespace}"
       parent_link="${namespace}/base_link"
@@ -144,6 +144,6 @@
       <box size="0.001 0.001 0.001" />
       <origin xyz="0.1 0 0" rpy="0 0 0" />
-  </xacro:camera_macro> -->
-  <xacro:include filename="$(find bearings)/description/camera_bebop2.xacro"/>
-  <xacro:camera_base namespace="${namespace}" ></xacro:camera_base>
+  </xacro:camera_macro>
+  <!-- <xacro:include filename="$(find bearings)/description/camera_bebop2.xacro"/>
+  <xacro:camera_base namespace="${namespace}" ></xacro:camera_base> -->
 </robot>

File: xacro/bebop2_3.xacro (robot description, xacro)
@@ -128,5 +128,5 @@
   </xacro:vertical_rotor>
  <!--Mount a Camera-->
-  <!-- <xacro:camera_macro
+  <xacro:camera_macro
       namespace="${namespace}"
       parent_link="${namespace}/base_link"
@@ -144,6 +144,6 @@
       <box size="0.001 0.001 0.001" />
       <origin xyz="0.1 0 0" rpy="0 0 0" />
-  </xacro:camera_macro> -->
-  <xacro:include filename="$(find bearings)/description/camera_bebop2.xacro"/>
-  <xacro:camera_base namespace="${namespace}" ></xacro:camera_base>
+  </xacro:camera_macro>
+  <!-- <xacro:include filename="$(find bearings)/description/camera_bebop2.xacro"/>
+  <xacro:camera_base namespace="${namespace}" ></xacro:camera_base> -->
 </robot>

File: xacro/bebop2_4.xacro (robot description, xacro)
@@ -128,5 +128,5 @@
   </xacro:vertical_rotor>
  <!--Mount a Camera-->
-  <!-- <xacro:camera_macro
+  <xacro:camera_macro
       namespace="${namespace}"
       parent_link="${namespace}/base_link"
@@ -144,6 +144,6 @@
       <box size="0.001 0.001 0.001" />
       <origin xyz="0.1 0 0" rpy="0 0 0" />
-  </xacro:camera_macro> -->
-  <xacro:include filename="$(find bearings)/description/camera_bebop2.xacro"/>
-  <xacro:camera_base namespace="${namespace}" ></xacro:camera_base>
+  </xacro:camera_macro>
+  <!-- <xacro:include filename="$(find bearings)/description/camera_bebop2.xacro"/>
+  <xacro:camera_base namespace="${namespace}" ></xacro:camera_base> -->
 </robot>

File: xacro/bebop2_5.xacro (robot description, xacro)
@@ -5,5 +5,5 @@
   <xacro:property name="rotor_velocity_slowdown_sim" value="10" />
   <xacro:property name="use_mesh_file" value="true" />
-  <xacro:property name="mesh_file" value="package://bearings/meshes/bebop2_1.dae" />
+  <xacro:property name="mesh_file" value="package://bearings/meshes/bebop2_5.dae" />
   <xacro:property name="mass" value="0.503" /> <!-- [kg] -->
   <xacro:property name="body_width" value="0.316618" /> <!-- [m] -->
@@ -141,8 +141,10 @@
       noise_mean="0.0"
       noise_stddev="0.007"
-      enable_visual="true">
+      enable_visual="true"
+      focal_length = "375">
       <box size="0.001 0.001 0.001" />
       <origin xyz="0.1 0 0" rpy="0 0 0" />
   </xacro:camera_macro>
+  <!-- focal_lengtth = image_width / (2*tan(hfov_radian / 2)> -->
   <!-- <xacro:include filename="$(find bearings)/description/camera_bebop2.xacro"/>
   <xacro:camera_base namespace="${namespace}" ></xacro:camera_base> -->
