Commit message: Added - Rotational Groudn Truth Added - Camera Calibration Modf - Cameras xacro for iris drone

File: description/camera_bebop2.xacro (robot description, xacro)
@@ -5,5 +5,5 @@
       <parent link="${namespace}/base_link"/>
       <child link="camera_link"/>
-      <origin xyz="0.11 0 0" rpy="0 0 0"/>
+      <origin xyz="0.113 0 0" rpy="0 0 0"/>
     </joint>
     <link name="camera_link">
@@ -24,102 +24,38 @@
       <material>Gazebo/Red</material>
       <sensor type="camera" name="camera">
-        <pose> 0 0 0 0 0 0 </pose>
+        <update_rate>30</update_rate>
         <visualize>false</visualize>
-        <update_rate>30</update_rate>
         <camera>
           <!-- <horizontal_fov>1.0472</horizontal_fov> -->
-          <horizontal_fov>2</horizontal_fov>
+          <!-- <horizontal_fov>2.09</horizontal_fov> -->
+          <!-- <horizontal_fov>2</horizontal_fov> -->
+          <!-- <horizontal_fov>1.6</horizontal_fov> -->
+          <!-- <horizontal_fov>1.75</horizontal_fov> -->
+          <!-- <horizontal_fov>1.3962634</horizontal_fov> -->
+          <!-- <horizontal_fov>0.3962634</horizontal_fov> -->
           <image>
-            <width>4096</width>
-            <height>3072</height>
+            <focal_length>700</focal_length>
+            <width>1920</width>
+            <height>1080</height>
             <format>R8G8B8</format>
           </image>
           <clip>
-            <near>0.01</near>
-            <far>150</far>
+            <near>0.02</near>
+            <far>300</far>
           </clip>
-          <noise>
-            <type>gaussian</type>
-            <!-- Noise is sampled independently per pixel on each frame.
+          <!-- <noise>
+            <type>gaussian</type> -->
+          <!-- Noise is sampled independently per pixel on each frame.
             That pixel's noise value is added to each of its color
             channels, which at that point lie in the range [0,1]. -->
-            <mean>0.0</mean>
-            <stddev>0.007</stddev>
-          </noise>
+          <!-- <mean>0.0</mean>
+            <stddev>0.003</stddev>
+          </noise> -->
           <lens>
             <intrinsics>
-              <fx>1505</fx>
-              <fy>1505</fy>
-              <cx>2048</cx>
-              <cy>1536</cy>
-              <s>0</s>
-            </intrinsics>
-          </lens>
-          <distortion>
-            <k1>0.14201146990975286</k1>
-            <k2>-0.19688011266332983</k2>
-            <k3>0.0429167931421525</k3>
-            <p1>-0.0054052167768174585</p1>
-            <p2>0.0011235413612189335</p2>
-          </distortion>
-        </camera>
-        <plugin name="camera_controller" filename="libgazebo_ros_camera.so">
-          <frame_name>camera_link_optical</frame_name>
-          <cameraName>camera_base</cameraName>
-        </plugin>
-      </sensor>
-    </gazebo>
-  </xacro:macro>
-  <xacro:macro name="camera_secondary" params="namespace">
-    <joint name="camera_under_joint" type="fixed">
-      <parent link="${namespace}/base_link"/>
-      <child link="camera_under_link"/>
-      <origin xyz="0 0 -0.04" rpy="0 ${pi/2} 0"/>
-    </joint>
-    <link name="camera_under_link">
-      <visual>
-        <geometry>
-          <box size="0.01 0.03 0.03"/>
-        </geometry>
-        <material name="Red"/>
-      </visual>
-    </link>
-    <joint name="camera_under_optical_joint" type="fixed">
-      <parent link="camera_under_link"/>
-      <child link="camera_under_link_optical"/>
-      <origin xyz="0 0 0" rpy="0 0 0"/>
-    </joint>
-    <link name="camera_under_link_optical"></link>
-    <gazebo reference="camera_under_link">
-      <material>Gazebo/Blue</material>
-      <sensor type="camera" name="camera">
-        <pose> 0 0 0 0 0 0 </pose>
-        <visualize>false</visualize>
-        <update_rate>30</update_rate>
-        <camera>
-          <horizontal_fov>2</horizontal_fov>
-          <image>
-            <width>752</width>
-            <height>480</height>
-            <format>R8G8B8</format>
-          </image>
-          <clip>
-            <near>0.01</near>            <!---->
-            <far>150</far>
-          </clip>
-          <noise>
-            <type>gaussian</type>
-            <!-- Noise is sampled independently per pixel on each frame.
-          That pixel's noise value is added to each of its color
-          channels, which at that point lie in the range [0,1]. -->
-            <mean>0.0</mean>
-            <stddev>0.007</stddev>
-          </noise>
-          <lens>
-            <intrinsics>
-              <fx>241.4268236</fx>
-              <fy>241.4268236</fy>
-              <cx>376</cx>
-              <cy>240</cy>
+              <fx>700</fx>
+              <fy>700</fy>
+              <cx>960</cx>
+              <cy>540</cy>
               <s>0</s>
             </intrinsics>
@@ -127,9 +63,80 @@
         </camera>
         <plugin name="camera_controller" filename="libgazebo_ros_camera.so">
-          <frame_name>camera_under_link_optical</frame_name>
-          <cameraName>camera_under_camera</cameraName>
+          <alwaysOn>true</alwaysOn>
+          <updateRate>0.0</updateRate>
+          <cameraName>camera_base</cameraName>
+          <cameraInfoTopicName>camera_info</cameraInfoTopicName>
+          <frameName>camera_link_optical</frameName>
+          <hackBaseline>0.07</hackBaseline>
+          <distortionK1>0.0</distortionK1>
+          <distortionK2>0.0</distortionK2>
+          <distortionK3>0.0</distortionK3>
+          <distortionT1>0.0</distortionT1>
+          <distortionT2>0.0</distortionT2>
         </plugin>
       </sensor>
     </gazebo>
-  </xacro:macro>
-</robot>
+    </xacro:macro>
+    <xacro:macro name="camera_secondary" params="namespace">
+      <joint name="camera_under_joint" type="fixed">
+        <parent link="${namespace}/base_link"/>
+        <child link="camera_under_link"/>
+        <origin xyz="0 0 -0.04" rpy="0 ${pi/2} 0"/>
+      </joint>
+      <link name="camera_under_link">
+        <visual>
+          <geometry>
+            <box size="0.01 0.03 0.03"/>
+          </geometry>
+          <material name="Red"/>
+        </visual>
+      </link>
+      <joint name="camera_under_optical_joint" type="fixed">
+        <parent link="camera_under_link"/>
+        <child link="camera_under_link_optical"/>
+        <origin xyz="0 0 0" rpy="0 0 0"/>
+      </joint>
+      <link name="camera_under_link_optical"></link>
+      <gazebo reference="camera_under_link">
+        <material>Gazebo/Blue</material>
+        <sensor type="camera" name="camera">
+          <pose> 0 0 0 0 0 0 </pose>
+          <visualize>false</visualize>
+          <update_rate>30</update_rate>
+          <camera>
+            <horizontal_fov>2</horizontal_fov>
+            <image>
+              <width>752</width>
+              <height>480</height>
+              <format>R8G8B8</format>
+            </image>
+            <clip>
+              <near>0.01</near>              <!---->
+              <far>150</far>
+            </clip>
+            <noise>
+              <type>gaussian</type>
+              <!-- Noise is sampled independently per pixel on each frame.
+          That pixel's noise value is added to each of its color
+          channels, which at that point lie in the range [0,1]. -->
+              <mean>0.0</mean>
+              <stddev>0.007</stddev>
+            </noise>
+            <lens>
+              <intrinsics>
+                <fx>241.4268236</fx>
+                <fy>241.4268236</fy>
+                <cx>376</cx>
+                <cy>240</cy>
+                <s>0</s>
+              </intrinsics>
+            </lens>
+          </camera>
+          <plugin name="camera_controller" filename="libgazebo_ros_camera.so">
+            <frame_name>camera_under_link_optical</frame_name>
+            <cameraName>camera_under_camera</cameraName>
+          </plugin>
+        </sensor>
+      </gazebo>
+    </xacro:macro>
+  </robot>

File: description/camera_iris.xacro (robot description, xacro)
@@ -5,5 +5,5 @@
       <parent link="${namespace}/base_link"/>
       <child link="camera_link"/>
-      <origin xyz="0.095 0 0" rpy="0 0 0"/>
+      <origin xyz="0.099 0 0" rpy="0 0 0"/>
     </joint>
     <link name="camera_link">
@@ -22,13 +22,18 @@
     <link name="camera_link_optical"></link>
     <gazebo reference="camera_link">
-      <material>Gazebo/Red</material>
+      <material>Gazebo/BlueGlow</material>
       <sensor type="camera" name="camera">
-        <pose> 0 0 0 0 0 0 </pose>
+        <update_rate>30</update_rate>
         <visualize>false</visualize>
-        <update_rate>30</update_rate>
         <camera>
           <!-- <horizontal_fov>1.0472</horizontal_fov> -->
+          <!-- <horizontal_fov>2.09</horizontal_fov> -->
           <!-- <horizontal_fov>2</horizontal_fov> -->
+          <!-- <horizontal_fov>1.6</horizontal_fov> -->
+          <!-- <horizontal_fov>1.75</horizontal_fov> -->
+          <!-- <horizontal_fov>1.3962634</horizontal_fov> -->
+          <!-- <horizontal_fov>0.3962634</horizontal_fov> -->
           <image>
+            <focal_length>700</focal_length>
             <width>1920</width>
             <height>1080</height>
@@ -36,15 +41,15 @@
           </image>
           <clip>
-            <near>0.01</near>            <!---->
-            <far>150</far>
+            <near>0.02</near>
+            <far>300</far>
           </clip>
-          <noise>
-            <type>gaussian</type>
+          <!-- <noise>
+            <type>gaussian</type> -->
             <!-- Noise is sampled independently per pixel on each frame.
             That pixel's noise value is added to each of its color
             channels, which at that point lie in the range [0,1]. -->
-            <mean>0.0</mean>
-            <stddev>0.007</stddev>
-          </noise>
+            <!-- <mean>0.0</mean>
+            <stddev>0.003</stddev>
+          </noise> -->
           <lens>
             <intrinsics>
@@ -58,6 +63,15 @@
         </camera>
         <plugin name="camera_controller" filename="libgazebo_ros_camera.so">
-          <frame_name>camera_link_optical</frame_name>
+          <alwaysOn>true</alwaysOn>
+          <updateRate>0.0</updateRate>
           <cameraName>camera_base</cameraName>
+          <cameraInfoTopicName>camera_info</cameraInfoTopicName>
+          <frameName>camera_link_optical</frameName>
+          <hackBaseline>0.07</hackBaseline>
+          <distortionK1>0.0</distortionK1>
+          <distortionK2>0.0</distortionK2>
+          <distortionK3>0.0</distortionK3>
+          <distortionT1>0.0</distortionT1>
+          <distortionT2>0.0</distortionT2>
         </plugin>
       </sensor>

File: xacro/iris1.xacro (robot description, xacro)
@@ -166,4 +166,4 @@
   <xacro:include filename="$(find bearings)/description/camera_iris.xacro"/>
   <xacro:camera_base namespace="${namespace}" ></xacro:camera_base>
-  <xacro:under_camera namespace="${namespace}" ></xacro:under_camera>
+  <!-- <xacro:under_camera namespace="${namespace}" ></xacro:under_camera> -->
 </robot>

File: xacro/iris2.xacro (robot description, xacro)
@@ -166,4 +166,4 @@
   <xacro:include filename="$(find bearings)/description/camera_iris.xacro"/>
   <xacro:camera_base namespace="${namespace}" ></xacro:camera_base>
-  <xacro:under_camera namespace="${namespace}" ></xacro:under_camera>
+  <!-- <xacro:under_camera namespace="${namespace}" ></xacro:under_camera> -->
 </robot>

File: xacro/iris3.xacro (robot description, xacro)
@@ -169,4 +169,4 @@
   <xacro:include filename="$(find bearings)/description/camera_iris.xacro"/>
   <xacro:camera_base namespace="${namespace}" ></xacro:camera_base>
-  <xacro:under_camera namespace="${namespace}" ></xacro:under_camera>
+  <!-- <xacro:under_camera namespace="${namespace}" ></xacro:under_camera> -->
 </robot>

File: xacro/iris4.xacro (robot description, xacro)
@@ -169,4 +169,4 @@
   <xacro:include filename="$(find bearings)/description/camera_iris.xacro"/>
   <xacro:camera_base namespace="${namespace}" ></xacro:camera_base>
-  <xacro:under_camera namespace="${namespace}" ></xacro:under_camera>
+  <!-- <xacro:under_camera namespace="${namespace}" ></xacro:under_camera> -->
 </robot>

File: xacro/iris5.xacro (robot description, xacro)
@@ -169,4 +169,4 @@
   <xacro:include filename="$(find bearings)/description/camera_iris.xacro"/>
   <xacro:camera_base namespace="${namespace}" ></xacro:camera_base>
-  <xacro:under_camera namespace="${namespace}" ></xacro:under_camera>
+  <!-- <xacro:under_camera namespace="${namespace}" ></xacro:under_camera> -->
 </robot>
